File: CurrentControl.sch (KiCad schematic (older format))
At the start: 7 parts, among them P1 CONN_01X01, Q401 BUK9575, U201 LMV358

Commit message: Updated part numbers and generated BOM
Parts:
- P1: value CONN_01X01 -> HEATSINK; MPN (none) -> FA-T220-38E
Changed lines of the file:
@@
 P 9350 3500
 F 0 "P1" H 9350 3600 50  0000 C CNN
-F 1 "CONN_01X01" V 9450 3500 50  0000 C CNN
+F 1 "HEATSINK" V 9450 3500 50  0000 C CNN
 F 2 "Current:FA-T220-38E" H 9350 3500 60  0001 C CNN
 F 3 "" H 9350 3500 60  0000 C CNN
+F 4 "FA-T220-38E" H 9350 3500 60  0001 C CNN "MPN"
 	1    9350 3500
 	1    0    0    -1
