File: PowerRegulation.sch (KiCad schematic (older format))
At the start: 6 parts, among them U301 LM2931D-R

Commit message: Updated part numbers and generated BOM
Parts:
- C301, C302: value C -> .1
- U301: value LM2931D-R -> LM2931; MPN (none) -> LM2931D-R
Changed lines of the file:
@@
 P 4000 3300
 F 0 "C301" H 4050 3400 50  0000 L CNN
-F 1 "C" H 4050 3200 50  0000 L CNN
+F 1 ".1" H 4050 3200 50  0000 L CNN
 F 2 "SMD_Packages:SMD-0805" H 4038 3150 30  0001 C CNN
 F 3 "" H 4000 3300 60  0000 C CNN
@@
 P 6200 3450
 F 0 "C302" H 6250 3550 50  0000 L CNN
-F 1 "C" H 6250 3350 50  0000 L CNN
+F 1 ".1" H 6250 3350 50  0000 L CNN
 F 2 "SMD_Packages:SMD-0805" H 6238 3300 30  0001 C CNN
 F 3 "" H 6200 3450 60  0000 C CNN
@@
 P 4750 3150
 F 0 "U301" H 5000 3000 60  0000 C CNN
-F 1 "LM2931D-R" H 4750 3800 60  0000 C CNN
+F 1 "LM2931" H 4750 3800 60  0000 C CIN
 F 2 "SMD_Packages:SOIC-8-N" H 4600 3150 60  0001 C CNN
 F 3 "" H 4600 3150 60  0000 C CNN
+F 4 "LM2931D-R" H 4750 3150 60  0001 C CNN "MPN"
 	1    4750 3150
 	1    0    0    -1
