File: VoltageControl.sch (KiCad schematic (older format))
At the start: 7 parts, among them U201 LMV358

Commit message: Updated part numbers and generated BOM
Parts:
- C201: value C -> .1
- D201: value DIODE -> 1N4148
- U201: MPN Value -> LMV358IDT
Changed lines of the file:
@@
 F 2 "SMD_Packages:SOIC-8-N" H 5850 3050 60  0001 C CNN
 F 3 "" H 5850 3050 60  0001 C CNN
-F 4 "Value" H 5850 3050 60  0001 C CNN "MPN"
+F 4 "LMV358IDT" H 5850 3050 60  0001 C CNN "MPN"
 	1    5850 3050
 	1    0    0    -1
@@
 P 5150 2400
 F 0 "C201" H 5200 2500 50  0000 L CNN
-F 1 "C" H 5200 2300 50  0000 L CNN
+F 1 ".1" H 5200 2300 50  0000 L CNN
 F 2 "SMD_Packages:SMD-0805" H 5188 2250 30  0001 C CNN
 F 3 "" H 5150 2400 60  0000 C CNN
@@
 P 6750 3050
 F 0 "D201" H 6750 3150 40  0000 C CNN
-F 1 "DIODE" H 6750 2950 40  0000 C CNN
+F 1 "1N4148" H 6750 2950 40  0000 C CNN
 F 2 "SMD_Packages:SOD-523" H 6750 3050 60  0001 C CNN
 F 3 "http://www.diodes.com/datasheets/ds30396.pdf" H 6750 3050 60  0001 C CNN
