File: CurrentSinkOrSwim.kicad_pcb (KiCad board)
At the start: 2 copper layers, 41.7 x 47.8 mm, 23 parts, among them P1 CONN_01X01, P101 CONN_01X02, P102 CONN_01X03, P103 CONN_01X02, Q401 BUK9575, U201 LMV358, U301 LM2931D-R

Commit message: Unknown changes before a Vagrant VM destroy
Parts:
- added REF**: MountingHole_3MM, Current:MountingHole_3MM, F.Cu at (149.9, 85.7)
- added REF**: MountingHole_3MM, Current:MountingHole_3MM, F.Cu at (149.9, 33.0)
- added REF**: MountingHole_3MM, Current:MountingHole_3MM, F.Cu at (104.1, 33.0)
Other:
- board size 41.7 x 47.8 mm -> 45.6 x 53.7 mm
Changed lines of the file:
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@@
-(kicad_pcb (version 4) (host pcbnew 0.201502010101+5397~21~ubuntu14.04.1-product)
+(kicad_pcb (version 4) (host pcbnew 0.201509151501+6198~30~ubuntu14.04.1-product)
   (general
-    (links 42)
+    (links 0)
     (no_connects 0)
-    (area 106.121999 35.763999 147.878001 83.616001)
+    (area 105.817599 35.434199 148.182401 89.152801)
     (thickness 1.6)
-    (drawings 5)
+    (drawings 6)
     (tracks 132)
     (zones 0)
-    (modules 23)
+    (modules 26)
     (nets 17)
   )
@@
     (mod_text_size 1 1)
     (mod_text_width 0.15)
-    (pad_size 1.5 1.5)
-    (pad_drill 0.6)
+    (pad_size 3 3)
+    (pad_drill 3)
     (pad_to_mask_clearance 0)
     (aux_axis_origin 0 0)
@@
     (add_net "Net-(P101-Pad1)")
     (add_net "Net-(Q401-PadS)")
+  )
+  (module Current:MountingHole_3MM (layer F.Cu)
+    (at 149.86 85.725)
+    (fp_text reference REF** (at 0 4) (layer F.SilkS) hide
+      (effects (font (size 1 1) (thickness 0.15)))
+    )
+    (fp_text value MountingHole_3MM (at 0 -4) (layer F.Fab) hide
+      (effects (font (size 1 1) (thickness 0.15)))
+    )
+    (fp_circle (center 0 0) (end 3 0) (layer Cmts.User) (width 0.15))
+    (pad "" np_thru_hole circle (at 0 0) (size 3 3) (drill 3) (layers *.Cu *.Mask F.SilkS))
+  )
+  (module Current:MountingHole_3MM (layer F.Cu)
+    (at 149.86 33.02)
+    (fp_text reference REF** (at 0 4) (layer F.SilkS) hide
+      (effects (font (size 1 1) (thickness 0.15)))
+    )
+    (fp_text value MountingHole_3MM (at 0 -4) (layer F.Fab) hide
+      (effects (font (size 1 1) (thickness 0.15)))
+    )
+    (fp_circle (center 0 0) (end 3 0) (layer Cmts.User) (width 0.15))
+    (pad "" np_thru_hole circle (at 0 0) (size 3 3) (drill 3) (layers *.Cu *.Mask F.SilkS))
   )
   (module SMD_Packages:SMD-0805 (layer B.Cu)
@@
   )
   (module Current:P090L-02F25BR10K (layer F.Cu)
+    (at 113.538 79.883)
+    (fp_text reference RV201 (at 5.969 0.635 90) (layer F.SilkS)
+      (effects (font (size 1.016 1.016) (thickness 0.15)))
+    )
+    (fp_text value 10K (at 0 -9.906) (layer F.Fab) hide
+      (effects (font (size 1.5 1.5) (thickness 0.15)))
+    )
+    (fp_line (start -1.778 3.556) (end -1.778 8.89) (layer Eco1.User) (width 0.15))
+    (fp_line (start -1.778 8.89) (end 2.54 8.89) (layer Eco1.User) (width 0.15))
+    (fp_line (start 2.54 8.89) (end 2.54 3.556) (layer Eco1.User) (width 0.15))
+    (fp_line (start -4.9 -5.9) (end 4.9 -5.9) (layer F.SilkS) (width 0.15))
+    (fp_line (start -4.9 3.5) (end 4.9 3.5) (layer F.SilkS) (width 0.15))
+    (fp_line (start 4.9 -5.9) (end 4.9 3.5) (layer F.SilkS) (width 0.15))
+    (fp_line (start -4.9 -5.9) (end -4.9 3.5) (layer F.SilkS) (width 0.15))
+    (pad 3 thru_hole circle (at 2.5 0) (size 2 2) (drill 1) (layers *.Cu *.Mask F.SilkS)
+      (net 2 GND))
+    (pad 2 thru_hole circle (at 0 0) (size 2 2) (drill 1) (layers *.Cu *.Mask F.SilkS)
+      (net 13 "Net-(R201-Pad2)"))
+    (pad 1 thru_hole circle (at -2.5 0) (size 2 2) (drill 1) (layers *.Cu *.Mask F.SilkS)
+      (net 15 "Net-(RV201-Pad1)"))
+    (pad "" np_thru_hole circle (at 5.1 -3.3) (size 2.2 2.2) (drill 2.2) (layers *.Cu *.Mask F.SilkS))
+    (pad "" np_thru_hole circle (at -5.1 -3.3) (size 2.2 2.2) (drill 2.2) (layers *.Cu *.Mask F.SilkS))
+  )
+  (module Current:P090L-02F25BR10K (layer F.Cu)
     (at 127.508 79.756)
     (fp_text reference RV401 (at 5.969 0.635 90) (layer F.SilkS)
@@
     (pad 1 thru_hole circle (at -2.5 0) (size 2 2) (drill 1) (layers *.Cu *.Mask F.SilkS)
       (net 14 "Net-(R401-Pad2)"))
-    (pad "" np_thru_hole oval (at 5.1 -3.3) (size 2 2.2) (drill oval 2 2.2) (layers *.Cu *.Mask F.SilkS))
-    (pad "" np_thru_hole oval (at -5.1 -3.3) (size 2 2.2) (drill oval 2 2.2) (layers *.Cu *.Mask F.SilkS))
-  )
-  (module Current:P090L-02F25BR10K (layer F.Cu)
-    (at 113.538 79.883)
-    (fp_text reference RV201 (at 5.969 0.635 90) (layer F.SilkS)
-      (effects (font (size 1.016 1.016) (thickness 0.15)))
-    )
-    (fp_text value 10K (at 0 -9.906) (layer F.Fab) hide
-      (effects (font (size 1.5 1.5) (thickness 0.15)))
-    )
-    (fp_line (start -1.778 3.556) (end -1.778 8.89) (layer Eco1.User) (width 0.15))
-    (fp_line (start -1.778 8.89) (end 2.54 8.89) (layer Eco1.User) (width 0.15))
-    (fp_line (start 2.54 8.89) (end 2.54 3.556) (layer Eco1.User) (width 0.15))
-    (fp_line (start -4.9 -5.9) (end 4.9 -5.9) (layer F.SilkS) (width 0.15))
-    (fp_line (start -4.9 3.5) (end 4.9 3.5) (layer F.SilkS) (width 0.15))
-    (fp_line (start 4.9 -5.9) (end 4.9 3.5) (layer F.SilkS) (width 0.15))
-    (fp_line (start -4.9 -5.9) (end -4.9 3.5) (layer F.SilkS) (width 0.15))
-    (pad 3 thru_hole circle (at 2.5 0) (size 2 2) (drill 1) (layers *.Cu *.Mask F.SilkS)
-      (net 2 GND))
-    (pad 2 thru_hole circle (at 0 0) (size 2 2) (drill 1) (layers *.Cu *.Mask F.SilkS)
-      (net 13 "Net-(R201-Pad2)"))
-    (pad 1 thru_hole circle (at -2.5 0) (size 2 2) (drill 1) (layers *.Cu *.Mask F.SilkS)
-      (net 15 "Net-(RV201-Pad1)"))
-    (pad "" np_thru_hole oval (at 5.1 -3.3) (size 2 2.2) (drill oval 2 2.2) (layers *.Cu *.Mask F.SilkS))
-    (pad "" np_thru_hole oval (at -5.1 -3.3) (size 2 2.2) (drill oval 2 2.2) (layers *.Cu *.Mask F.SilkS))
-  )
+    (pad "" np_thru_hole circle (at 5.1 -3.3) (size 2.2 2.2) (drill 2.2) (layers *.Cu *.Mask F.SilkS))
+    (pad "" np_thru_hole circle (at -5.1 -3.3) (size 2.2 2.2) (drill 2.2) (layers *.Cu *.Mask F.SilkS))
+  )
+  (module Current:MountingHole_3MM (layer F.Cu)
+    (at 104.14 33.02)
+    (fp_text reference REF** (at 0 4) (layer F.SilkS) hide
+      (effects (font (size 1 1) (thickness 0.15)))
+    )
+    (fp_text value MountingHole_3MM (at 0 -4) (layer F.Fab) hide
+      (effects (font (size 1 1) (thickness 0.15)))
+    )
+    (fp_circle (center 0 0) (end 3 0) (layer Cmts.User) (width 0.15))
+    (pad "" np_thru_hole circle (at 0 0) (size 3 3) (drill 3) (layers *.Cu *.Mask F.SilkS))
+  )
+  (gr_line (start 151.765 29.845) (end 151.765 46.99) (layer Edge.Cuts) (width 0.1))
   (gr_text "Current Sink\nOr Swim" (at 126.746 44.577) (layer F.SilkS)
     (effects (font (size 1.5 1.5) (thickness 0.3)))
